File: Timsah_Remote-Control/Timsah_Remote-Control.sch (KiCad schematic (older format))
At the start: 22 parts, among them IC1 PIC18F45K22-I_P, J1 Güç Girişi, J2 ICSP, J3 Klemens, SW1 SW, SW2 POWER SW, U1 MAX485E, U2 LM7805_TO220, U3 Joystick-A, U4 Joystick-B

Commit message: Remote controller schematic update.
- Some titels fixed
- Microcontroller updated
- Project library edited
- Some oriantations changed
Parts:
- removed IC1: PIC18F45K22-I_P, DIP1543W58P254L5175H635Q40N, symbol PIC18F45K22-I_P:PIC18F45K22-I_P
- removed U3: Joystick-A, symbol Timsah:Joystick
- removed U4: Joystick-B, symbol Timsah:Joystick
- added U3: PIC18F45K22-IP, Package_DIP:DIP-42_W15.24mm_LongPads, symbol Symols:PIC18F45K22-IP
- added U4: Joystick A, symbol Symols:Joystick
- added U5: Joystick B, symbol Symols:Joystick
- SW1: value SW -> Lights
Connections:
- net labels removed: Vin
- wire segments 90 -> 94
- no-connect marks 0 -> 28
Other:
- note added: "Güç"
- note added: "Motor Kontrolü"
- note added: "RS-485 Haberleşmesi"
- note added: "Sigorta"
- note removed: "Gerilim Düzenleyici ve Sigorta"
- note removed: "Güç Girişi"
- note removed: "Motor Kontrolleri"
- note removed: "RS-485 Haberleşme"
- moved on the sheet: F1, J1, POT1, R1, R4, R5, SW2A

Commit message: Added special controls.
Parts:
- added R10, R11, R12, R13, R14, R8, R9: 4k7, symbol Device:R
- added SW10: Backward, symbol Switch:SW_Push
- added SW3: Up, symbol Switch:SW_Push
- added SW4: Down, symbol Switch:SW_Push
- added SW5: Oto Depth, symbol Switch:SW_DPDT_x2
- added SW6: Turn Back, symbol Switch:SW_Push
- added SW7: Forward, symbol Switch:SW_Push
- added SW8: Right, symbol Switch:SW_Push
- added SW9: Left, symbol Switch:SW_Push
- R2: value 10K -> 4k7
- R3: value 100 -> 4k7
Connections:
- net +5V: now also SW1.1 (A), SW10.2, SW3.2, SW4.2, SW5.3 (C), SW6.2, SW7.2, SW8.2, SW9.2; no longer R3.1
- net GND: now also R3.2, R10.2, R11.2, R12.2, R13.2, R14.2, R8.2, R9.2
- net Forward: now reaches U3.19 (RD0/SCL2/SCK2/AN20)
- net Forward: now also R11.1, SW7.1
- net Right: now reaches U3.20 (RD1/SDI1/SDA2/CCP4/AN21)
- net Right: now also R12.1, SW8.1
- net Left: now reaches U3.21 (RD2/P2B/AN22)
- net Left: now also R13.1, SW9.1
- net Backward: now reaches U3.22 (RD3/P2C/~SS~2/AN23)
- net Backward: now also R14.1, SW10.1
- net Up: now reaches U3.27 (RD4/P2D/SDO2/AN24)
- net Up: now also R3.1, SW3.1
- net Down: now reaches U3.28 (RD5/P1B/AN25)
- net Down: now also R8.1, SW4.1
- net TURN_BACK: now reaches U3.29 (RD6/TX2/CK2/P1C/AN26)
- net TURN_BACK: now also R10.1, SW6.1
- net OTO_DEPTH: now reaches U3.30 (RD7/RX2/DT2/P1D/AN27)
- net OTO_DEPTH: now also R9.1, SW5.2 (B)
- no-connect marks 28 -> 21
Other:
- note added: "180 derece Geri Dönme"
- note added: "Derinlik Ayarı"
- note added: "Yön Kontrolü:\n15 derece sağ veya sola dönme\n1 saniye ileri veya geri gitme"
- note added: "Özel Kontroller"
- moved on the sheet: R1, R2, SW1A, U3

Commit message: Update schematics.
Parts:
- added POT2: 10K, symbol Device:R_POT
Connections:
- net +5V: now also POT2.1
- net GND: now also POT2.3
- net SERVO_Grip: now reaches U3.18 (RC3/SCL1/SCK1/AN15)
- net SERVO_Grip: now also POT2.2
- net SERVO renamed SERVO_Cam
- no-connect marks 21 -> 20
Other:
- note added: "Servo Kontrolü"
- note removed: "Kamera Yön Kontrolü"
- moved on the sheet: POT1, R2, SW1A
Changed lines of the file:
@@
 L Device:R_POT POT1
 U 1 1 5CBC8739
-P 7500 1200
-F 0 "POT1" H 7430 1246 50  0000 R CNN
-F 1 "10K" H 7430 1155 50  0000 R CNN
-F 2 "" H 7500 1200 50  0001 C CNN
-F 3 "~" H 7500 1200 50  0001 C CNN
-	1    7500 1200
-	1    0    0    -1
-$EndComp
-Text GLabel 7900 1200 2    50   Input ~ 0
-SERVO
-Wire Wire Line
-	7900 1200 7650 1200
+P 6950 1200
+F 0 "POT1" H 6880 1246 50  0000 R CNN
+F 1 "10K" H 6880 1155 50  0000 R CNN
+F 2 "" H 6950 1200 50  0001 C CNN
+F 3 "~" H 6950 1200 50  0001 C CNN
+	1    6950 1200
+	1    0    0    -1
+$EndComp
 $Comp
 L power:GND #PWR012
 U 1 1 5CBC891D
-P 7500 1500
-F 0 "#PWR012" H 7500 1250 50  0001 C CNN
-F 1 "GND" H 7505 1327 50  0000 C CNN
-F 2 "" H 7500 1500 50  0001 C CNN
-F 3 "" H 7500 1500 50  0001 C CNN
-	1    7500 1500
-	1    0    0    -1
-$EndComp
-Wire Wire Line
-	7500 1500 7500 1350
+P 6950 1500
+F 0 "#PWR012" H 6950 1250 50  0001 C CNN
+F 1 "GND" H 6955 1327 50  0000 C CNN
+F 2 "" H 6950 1500 50  0001 C CNN
+F 3 "" H 6950 1500 50  0001 C CNN
+	1    6950 1500
+	1    0    0    -1
+$EndComp
+Wire Wire Line
+	6950 1500 6950 1350
 $Comp
 L power:+5V #PWR011
 U 1 1 5CBC8A80
-P 7500 950
-F 0 "#PWR011" H 7500 800 50  0001 C CNN
-F 1 "+5V" H 7515 1123 50  0000 C CNN
-F 2 "" H 7500 950 50  0001 C CNN
-F 3 "" H 7500 950 50  0001 C CNN
-	1    7500 950
-	1    0    0    -1
-$EndComp
-Wire Wire Line
-	7500 950  7500 1050
+P 6950 950
+F 0 "#PWR011" H 6950 800 50  0001 C CNN
+F 1 "+5V" H 6965 1123 50  0000 C CNN
+F 2 "" H 6950 950 50  0001 C CNN
+F 3 "" H 6950 950 50  0001 C CNN
+	1    6950 950
+	1    0    0    -1
+$EndComp
+Wire Wire Line
+	6950 950  6950 1050
 Text GLabel 1300 2650 0    50   Input ~ 0
-SERVO
+SERVO_Cam
 Text Notes 7000 2100 0    79   ~ 16
-Kamera Yön Kontrolü
+Servo Kontrolü
 Wire Notes Line
 	11200 500  8400 500
@@
 	8350 500  8350 2150
 Wire Notes Line
-	8350 2150 6950 2150
-Wire Notes Line
-	6950 2150 6950 500
-Wire Notes Line
-	6950 500  8350 500
+	8350 2150 6650 2150
+Wire Notes Line
+	6650 2150 6650 500
+Wire Notes Line
+	6650 500  8350 500
 Text GLabel 4200 2450 2    50   Input ~ 0
 VRX-A
@@
 L power:GND #PWR06
 U 1 1 5CBCA853
-P 5550 1350
-F 0 "#PWR06" H 5550 1100 50  0001 C CNN
-F 1 "GND" H 5555 1177 50  0000 C CNN
-F 2 "" H 5550 1350 50  0001 C CNN
-F 3 "" H 5550 1350 50  0001 C CNN
-	1    5550 1350
+P 5350 1300
+F 0 "#PWR06" H 5350 1050 50  0001 C CNN
+F 1 "GND" H 5355 1127 50  0000 C CNN
+F 2 "" H 5350 1300 50  0001 C CNN
+F 3 "" H 5350 1300 50  0001 C CNN
+	1    5350 1300
 	1    0    0    -1
 $EndComp
@@
 L power:+5V #PWR010
 U 1 1 5CBCA8C0
-P 6650 900
-F 0 "#PWR010" H 6650 750 50  0001 C CNN
-F 1 "+5V" H 6665 1073 50  0000 C CNN
-F 2 "" H 6650 900 50  0001 C CNN
-F 3 "" H 6650 900 50  0001 C CNN
-	1    6650 900
+P 6450 850
+F 0 "#PWR010" H 6450 700 50  0001 C CNN
+F 1 "+5V" H 6465 1023 50  0000 C CNN
+F 2 "" H 6450 850 50  0001 C CNN
+F 3 "" H 6450 850 50  0001 C CNN
+	1    6450 850
 	1    0    0    -1
 $EndComp
@@
 L Device:R R2
 U 1 1 5CBCA902
-P 5850 1150
-F 0 "R2" V 5750 1150 50  0000 C CNN
-F 1 "4k7" V 5850 1150 50  0000 C CNN
-F 2 "" V 5780 1150 50  0001 C CNN
-F 3 "~" H 5850 1150 50  0001 C CNN
-	1    5850 1150
-	0    1    1    0
-$EndComp
-Wire Wire Line
-	5550 1350 5550 1150
-Wire Wire Line
-	5550 1150 5700 1150
-Wire Wire Line
-	6050 1150 6000 1150
-Text GLabel 6050 1400 3    50   Input ~ 0
+P 5650 1100
+F 0 "R2" V 5550 1100 50  0000 C CNN
+F 1 "4k7" V 5650 1100 50  0000 C CNN
+F 2 "" V 5580 1100 50  0001 C CNN
+F 3 "~" H 5650 1100 50  0001 C CNN
+	1    5650 1100
+	0    1    1    0
+$EndComp
+Wire Wire Line
+	5350 1300 5350 1100
+Wire Wire Line
+	5350 1100 5500 1100
+Wire Wire Line
+	5850 1100 5800 1100
+Text GLabel 5850 1350 3    50   Input ~ 0
 SW
 Wire Wire Line
-	6050 1400 6050 1150
+	5850 1350 5850 1100
 Text GLabel 4200 1750 2    50   Input ~ 0
 SW
 Wire Notes Line
-	6900 2150 6900 500
+	6600 2150 6600 500
 Wire Notes Line
 	5200 500  5200 2150
 Wire Notes Line
-	5200 500  6900 500
-Wire Notes Line
-	5200 2150 6900 2150
-Text Notes 5450 2100 0    79   ~ 16
+	5200 500  6600 500
+Wire Notes Line
+	5200 2150 6600 2150
+Text Notes 5250 2100 0    79   ~ 16
 Araç Ön Aydınlatması
 $Comp
 L Switch:SW_DPDT_x2 SW1
 U 1 1 5CBCD299
-P 6300 1150
-F 0 "SW1" H 6300 1350 50  0000 C CNN
-F 1 "Lights" H 6300 900 50  0000 C CNN
-F 2 "" H 6300 1150 50  0001 C CNN
-F 3 "" H 6300 1150 50  0001 C CNN
-	1    6300 1150
-	1    0    0    -1
-$EndComp
-Wire Wire Line
-	6100 1150 6050 1150
-Connection ~ 6050 1150
+P 6100 1100
+F 0 "SW1" H 6100 1300 50  0000 C CNN
+F 1 "Lights" H 6100 850 50  0000 C CNN
+F 2 "" H 6100 1100 50  0001 C CNN
+F 3 "" H 6100 1100 50  0001 C CNN
+	1    6100 1100
+	1    0    0    -1
+$EndComp
+Wire Wire Line
+	5900 1100 5850 1100
+Connection ~ 5850 1100
 $Comp
 L Regulator_Linear:LM7805_TO220 U2
@@
 	6800 2600 7200 2600
 NoConn ~ 6800 2800
-NoConn ~ 6500 1250
+NoConn ~ 6300 1200
 NoConn ~ 1400 1150
 NoConn ~ 1400 1250
@@
 NoConn ~ 1400 2450
 NoConn ~ 1400 2550
-NoConn ~ 1400 2750
 NoConn ~ 1400 2850
 NoConn ~ 1400 2950
@@
 Sigorta
 Wire Wire Line
-	6650 900  6650 1050
-Wire Wire Line
-	6650 1050 6500 1050
+	6450 850  6450 1000
+Wire Wire Line
+	6450 1000 6300 1000
 $Comp
 L power:GND #PWR023
@@
 Text Notes 2350 7550 0    79   ~ 16
 Özel Kontroller
+$Comp
+L Device:R_POT POT2
+U 1 1 5D2A70BC
+P 7750 1200
+F 0 "POT2" H 7680 1246 50  0000 R CNN
+F 1 "10K" H 7680 1155 50  0000 R CNN
+F 2 "" H 7750 1200 50  0001 C CNN
+F 3 "~" H 7750 1200 50  0001 C CNN
+	1    7750 1200
+	1    0    0    -1
+$EndComp
+$Comp
+L power:GND #PWR038
+U 1 1 5D2A70C8
+P 7750 1500
+F 0 "#PWR038" H 7750 1250 50  0001 C CNN
+F 1 "GND" H 7755 1327 50  0000 C CNN
+F 2 "" H 7750 1500 50  0001 C CNN
+F 3 "" H 7750 1500 50  0001 C CNN
+	1    7750 1500
+	1    0    0    -1
+$EndComp
+Wire Wire Line
+	7750 1500 7750 1350
+$Comp
+L power:+5V #PWR037
+U 1 1 5D2A70D3
+P 7750 950
+F 0 "#PWR037" H 7750 800 50  0001 C CNN
+F 1 "+5V" H 7765 1123 50  0000 C CNN
+F 2 "" H 7750 950 50  0001 C CNN
+F 3 "" H 7750 950 50  0001 C CNN
+	1    7750 950
+	1    0    0    -1
+$EndComp
+Wire Wire Line
+	7750 950  7750 1050
+Text GLabel 1300 2750 0    50   Input ~ 0
+SERVO_Grip
+Wire Wire Line
+	1300 2750 1400 2750
+Text GLabel 8050 1050 1    50   Input ~ 0
+SERVO_Grip
+Wire Wire Line
+	8050 1050 8050 1200
+Wire Wire Line
+	7900 1200 8050 1200
+Wire Wire Line
+	7300 1050 7300 1200
+Wire Wire Line
+	7100 1200 7300 1200
+Text GLabel 7300 1050 1    50   Input ~ 0
+SERVO_Cam
 $EndSCHEMATC

Commit message: Schematic updates.
Parts:
- removed J1: Güç Girişi, symbol Connector:Conn_01x02_Female
- added J1: Güç Girişi, symbol Connector:Conn_01x03_Male
- added R15, R16, R17: 10k, symbol Device:R
- R4, R5: value 20K -> 20k
Connections:
- net +5V: now also R15.1, R16.1, R17.1
- net ENABLE: now also R16.2
- net GND: now also SW1.3 (C), SW5.1 (A), J1.1 (Pin_1), J1.3 (Pin_3); no longer R2.2, R9.2
- net OTO_DEPTH: now also R9.2; no longer R9.1, SW5.2 (B)
- net RX1: now also R15.2
- net SW: now also R2.2; no longer R2.1, SW1.2 (B)
- net TX1: now also R17.2
- net at SW2.2 (B): now also J1.2 (Pin_2)
- new net: R2.1, SW1.2 (B)
- new net: R9.1, SW5.2 (B)
- no-connect marks 20 -> 18
Other:
- moved on the sheet: J3, R2, R4, R5, R6, SW1A, U1

Commit message: Remote update.
- PCB design started.
Parts:
- removed SW1: Lights, symbol Switch:SW_DPDT_x2
- removed SW2: POWER SW, symbol Switch:SW_DPDT_x2
- removed SW5: Oto Depth, symbol Switch:SW_DPDT_x2
- added SW1: Oto Depth, Timsah_Remote-Control:SW_Slide_1P2T_0.105pitch, symbol Switch:SW_Push_SPDT
- added SW2: Lights, Timsah_Remote-Control:SW_Slide_1P2T_0.105pitch, symbol Switch:SW_Push_SPDT
- added SW5: Power, Timsah_Remote-Control:SW_Slide_1P2T_0.105pitch, symbol Switch:SW_Push_SPDT
- C1, C2: footprint (none) -> Capacitor_THT:C_Radial_D5.0mm_H7.0mm_P2.00mm
- D1: footprint (none) -> LED_THT:LED_D5.0mm
- F1: footprint (none) -> Timsah_Remote-Control:Fuseholder_23x9x10mm
- J1: footprint (none) -> Connector_PinHeader_2.54mm:PinHeader_1x03_P2.54mm_Vertical
- J2: footprint (none) -> Connector_PinHeader_2.54mm:PinHeader_1x05_P2.54mm_Vertical
- J3: footprint (none) -> TerminalBlock_4Ucon:TerminalBlock_4Ucon_1x02_P3.50mm_Vertical
- POT1, POT2: footprint (none) -> Timsah_Remote-Control:Potentiometer_Lineer-B503
- R1, R10, R11, R12, R13, R14, R15, R16, R17, R2, R3, R4, R5, R6, R7, R8, R9: footprint (none) -> Resistor_THT:R_Axial_DIN0207_L6.3mm_D2.5mm_P10.16mm_Horizontal
- SW10, SW3, SW4, SW6, SW7, SW8, SW9: footprint (none) -> Button_Switch_THT:SW_PUSH_6mm_H5mm
- U1: footprint (none) -> Package_DIP:DIP-8_W7.62mm_Socket
- U3: footprint Package_DIP:DIP-42_W15.24mm_LongPads -> Package_DIP:DIP-40_W15.24mm_Socket
- U4, U5: footprint (none) -> Timsah_Remote-Control:Joystick
Connections:
- net +5V: now also SW1.3 (C), SW2.1 (A)
- net GND: now also SW1.1 (A), SW2.3 (C)
- net at R2.1: now also SW2.2 (B)
- net at F1.2: now also SW5.1 (A)
- net at J1.2 (Pin_2): now also SW5.2 (B)
- net at R9.1: now also SW1.2 (B)
