File: Timsah_Main_Board/Timsah_Main_Board.sch (KiCad schematic (older format))
At the start: 1 part

Commit message: Initialize Schematic
Parts:
- added J?: SAG, symbol Connector:Screw_Terminal_01x03
- added J?: SOL, symbol Connector:Screw_Terminal_01x03
- added J?: UST_1, symbol Connector:Screw_Terminal_01x03
- added J?: UST_2, symbol Connector:Screw_Terminal_01x03
- added J? (x3): JSN-SR04T, symbol Connector:Conn_01x04_Female
- added R? (x2): 10k, symbol Device:R
- added U?: PIC18F45K22-IP, Package_DIP:DIP-42_W15.24mm_LongPads, symbol Symols:PIC18F45K22-IP
Connections:
- net at U?.1 (~MCLR~/VPP/RE3): now also R?.2
- net +5V: now reaches U?.11 (VDD)
- net +5V: now also U?.32 (VDD), J?.1 (Pin_1), J?.1 (Pin_1), J?.1 (Pin_1), R?.1, R?.1, U?.11 (VDD), U?.32 (VDD)
- net GND: now reaches U?.12 (VSS)
- net GND: now also U?.31 (VSS), J?.2 (Pin_2), J?.2 (Pin_2), J?.2 (Pin_2), J?.2 (Pin_2), J?.4 (Pin_4), J?.4 (Pin_4), J?.4 (Pin_4), U?.12 (VSS), U?.31 (VSS)
- net PWM1: now reaches U?.17 (RC2/CTPLS/CCP1/P1A/T5CKI/AN14)
- net PWM1: now also J?.1 (Pin_1)
- net PWM4: now reaches U?.20 (RD1/SDI1/SDA2/CCP4/AN21)
- net PWM4: now also J?.1 (Pin_1)
- net PWM2: now reaches U?.36 (AN9/C12IN2-/CTED2/CCP2/RB3)
- net PWM2: now also J?.1 (Pin_1)
- net PWM3: now reaches U?.38 (AN13/CCP3/T1G/IOC/CCP3/RB5)
- net PWM3: now also J?.1 (Pin_1)
- new net: R?.2, U?.1 (~MCLR~/VPP/RE3)
- new net BEC1: J?.3 (Pin_3), J?.3 (Pin_3), J?.3 (Pin_3), J?.3 (Pin_3)
- new net ECHO1: J?.3 (Pin_3), U?.22 (RD3/P2C/~SS~2/AN23)
- new net ECHO2: J?.3 (Pin_3), U?.27 (RD4/P2D/SDO2/AN24)
- new net ECHO3: J?.3 (Pin_3), U?.28 (RD5/P1B/AN25)
- new net TRIG1: J?.2 (Pin_2), U?.19 (RD0/SCL2/SCK2/AN20)
- new net TRIG2: J?.2 (Pin_2), U?.20 (RD1/SDI1/SDA2/CCP4/AN21)
- new net TRIG3: J?.2 (Pin_2), U?.21 (RD2/P2B/AN22)
Other:
- note added: "ESC Bağlantıları"
- note added: "JSN-SR04T Ultrasonik Sensörler"
- moved on the sheet: U?

Commit message: Update Main Board.
Parts:
- added C1, C5, C6: 0.1uF, symbol Device:C_Small
- added C2, C3, C4: 1uF, symbol Device:C_Small
- added D1: PWR, symbol Device:LED
- added F1, F2: 5A, symbol Device:Fuse
- added J12: Raspberry_PWR, symbol Connector:Screw_Terminal_01x03
- added J13: Jetson_PWR, symbol Connector:Screw_Terminal_01x03
- added J14: RS485, symbol Connector:Screw_Terminal_01x02
- added J15: PWR_IN, symbol Connector:Screw_Terminal_01x02
- added J2: ICSP_Main, symbol Connector:Conn_01x06_Male
- added J5: MPU9250, symbol Connector:Conn_01x10_Female
- added J6: MS5803-14BA, symbol Connector:Conn_01x07_Female
- added J8: ICSP_Slave, symbol Connector:Conn_01x06_Male
- added R10, R9: 20k, symbol Device:R
- added R11, R7: 270, symbol Device:R
- added R12: 120, symbol Device:R
- added R13, R8: 820, symbol Device:R
- added R3: 1k, symbol Device:R
- added R4, R5, R6: 10k, symbol Device:R
- added SW1: PWR, symbol Switch:SW_SPDT
- added U3: AMS1117-3.3, Package_TO_SOT_SMD:SOT-223-3_TabPin2, symbol Regulator_Linear:AMS1117-3.3
- added U4, U6: LM338, Package_TO_SOT_THT:TO-3, symbol Symols:LM338
- added U5: MAX485E, symbol Interface_UART:MAX485E
- gave numbers to parts that had none: 11
Connections:
- net +5V: now also C3.1, C4.1, J12.1 (Pin_1), J2.2 (Pin_2), J5.10 (Pin_10), J8.2 (Pin_2), R10.2, R11.1, R4.1, R5.1, R6.1, U3.3 (VI), U5.8 (VCC), U6.2 (VO)
- net GND: now also C1.2, C2.2, C3.2, C4.2, C5.2, C6.2, D1.1 (K), J12.3 (Pin_3), J13.3 (Pin_3), J15.2 (Pin_2), J2.3 (Pin_3), J5.1 (Pin_1), J5.4 (Pin_4), J5.9 (Pin_9), J6.1 (Pin_1), J6.6 (Pin_6), J8.3 (Pin_3), R13.2, R8.2, R9.1, U3.1 (GND), U5.5 (GND)
- net TRIG1: now also U2.2 (AN0/C12IN0-/RA0); no longer U2.19 (RD0/SCL2/SCK2/AN20)
- net TRIG2: now also U2.3 (AN1/C12IN1-/RA1); no longer U2.20 (RD1/SDI1/SDA2/CCP4/AN21)
- net TRIG3: now also U2.4 (DACOUT/VREF-/AN2/C2IN+/RA2); no longer U2.21 (RD2/P2B/AN22)
- net ~MCLR1: now reaches R1.2, U1.1 (~MCLR~/VPP/RE3)
- net ~MCLR1: now also J2.1 (Pin_1)
- net SCL: now reaches U1.18 (RC3/SCL1/SCK1/AN15)
- net SCL: now also U2.18 (RC3/SCL1/SCK1/AN15), J5.8 (Pin_8)
- net SDA: now reaches U1.23 (RC4/SDA1/SDI1/AN16)
- net SDA: now also U2.23 (RC4/SDA1/SDI1/AN16), J5.7 (Pin_7)
- net TX: now reaches U1.25 (RC6/TX1/CK1/AN18)
- net TX: now also R4.2, U5.4 (DI)
- net RX: now reaches U1.26 (RC7/RX1/DT1/AN19)
- net RX: now also R6.2, U5.1 (RO)
- net ENABLE: now reaches U1.3 (AN1/C12IN1-/RA1)
- net ENABLE: now also R5.2, U5.2 (~RE), U5.3 (DE)
- net PGC1: now reaches U1.39 (PGC/IOC/RB6)
- net PGC1: now also J2.5 (Pin_5)
- net PGD1: now reaches U1.40 (PGD/IOC/RB7)
- net PGD1: now also J2.4 (Pin_4)
- net ~MCLR2: now reaches R2.2, U2.1 (~MCLR~/VPP/RE3)
- net ~MCLR2: now also J8.1 (Pin_1)
- net INT: now reaches U2.15 (RC0/P2B/SOSCO/T1CKI/T3CKI/T3G)
- net INT: now also J5.3 (Pin_3)
- net PGC2: now reaches U2.39 (PGC/IOC/RB6)
- net PGC2: now also J8.5 (Pin_5)
- net PGD2: now reaches U2.40 (PGD/IOC/RB7)
- net PGD2: now also J8.4 (Pin_4)
- new net: R7.2, R8.1, U4.1 (ADJ)
- new net: C5.1, F1.1, U4.3 (VI)
- new net: F1.2, F2.2, SW1.1 (A)
- new net: J15.1 (Pin_1), SW1.2 (B)
- new net: D1.2 (A), R3.2
- new net: R11.2, R13.1, U6.1 (ADJ)
- new net: C6.1, F2.1, U6.3 (VI)
- new net: J14.2 (Pin_2), R10.1, R12.2, U5.6 (A)
- new net: J14.1 (Pin_1), R12.1, R9.2, U5.7 (B)
- new net +3V3: C1.1, J6.2 (Pin_2), U3.2 (VO)
- new net 5V-NANO: C2.1, J13.1 (Pin_1), R3.1, R7.1, U4.2 (VO)
- new net SCL2: J6.4 (Pin_4), U2.19 (RD0/SCL2/SCK2/AN20)
- new net SDA2: J6.3 (Pin_3), U2.20 (RD1/SDI1/SDA2/CCP4/AN21)
- no-connect marks 0 -> 56
Other:
- note added: "9 Eksen MEMS Sensörü"
- note added: "Ana Mikrodenetleyici"
- note added: "Basınç Sensörü"
- note added: "Güç"
- note added: "Güç Çıkışı"
- note added: "ICSP"
- note added: "RS-485 Haberleşmesi"
- note added: "Ultrasonik Sensörler"
- note added: "Yardımcı Mikrodenetleyici"
- note removed: "JSN-SR04T Ultrasonik Sensörler"
- moved on the sheet: J1, J10, J11, J3, J4, J7, J9, R1, R2, U1, U2

Commit message: Schematic Update
Parts:
- added J16: Jetson_I2C, symbol Connector:Conn_01x02_Male
- added J17: Servo, symbol Connector:Conn_01x03_Female
Connections:
- net BEC1: no longer J10.3 (Pin_3), J4.3 (Pin_3), J9.3 (Pin_3)
- net GND: now also J17.3 (Pin_3)
- net SCL: now also J16.1 (Pin_1)
- net SDA: now also J16.2 (Pin_2)
- net SERVO: now reaches U2.17 (RC2/CTPLS/CCP1/P1A/T5CKI/AN14)
- net SERVO: now also J17.1 (Pin_1)
- new net BEC2: J9.3 (Pin_3)
- new net BEC3: J17.2 (Pin_2), J4.3 (Pin_3)
- new net BEC4: J10.3 (Pin_3)
- no-connect marks 56 -> 55
Other:
- note added: "I2C\nHaberleşmesi"
- note added: "Servo\nKontrolü"
- moved on the sheet: J2, J8
Changed lines of the file:
@@
 	6100 1250 6150 1250
 Text GLabel 4950 1350 0    50   Input ~ 0
-BEC1
+BEC3
 Text GLabel 6100 950  0    50   Input ~ 0
-BEC1
+BEC2
 Text GLabel 6100 1350 0    50   Input ~ 0
-BEC1
+BEC4
 Wire Wire Line
 	6100 950  6150 950
@@
 Text Notes 5100 1700 0    100  ~ 20
 ESC Bağlantıları
-Text GLabel 900  2600 0    50   Input ~ 0
-PWM1
-Wire Wire Line
-	900  2600 1000 2600
-Text GLabel 3800 2700 2    50   Input ~ 0
-PWM2
-Wire Wire Line
-	3800 2700 3700 2700
-Text GLabel 3800 2900 2    50   Input ~ 0
-PWM3
-Wire Wire Line
-	3800 2900 3700 2900
-Text GLabel 900  1600 0    50   Input ~ 0
-PWM4
-Wire Wire Line
-	900  1600 1000 1600
 $Comp
 L Connector:Conn_01x04_Female J11
@@
 L Connector:Conn_01x06_Male J2
 U 1 1 5D05755B
-P 5150 3850
-F 0 "J2" V 5212 4094 50  0000 L CNN
-F 1 "ICSP_Main" V 5100 3650 50  0000 L CNN
-F 2 "" H 5150 3850 50  0001 C CNN
-F 3 "~" H 5150 3850 50  0001 C CNN
-	1    5150 3850
+P 5150 3350
+F 0 "J2" V 5212 3594 50  0000 L CNN
+F 1 "ICSP_Main" V 5100 3150 50  0000 L CNN
+F 2 "" H 5150 3350 50  0001 C CNN
+F 3 "~" H 5150 3350 50  0001 C CNN
+	1    5150 3350
 	0    -1   1    0
 $EndComp
@@
 Wire Wire Line
 	3700 3100 3800 3100
-Text GLabel 5350 4150 3    50   Input ~ 0
+Text GLabel 5350 3550 3    50   Input ~ 0
 PGC1
-Text GLabel 5250 4150 3    50   Input ~ 0
+Text GLabel 5250 3550 3    50   Input ~ 0
 PGD1
-Text GLabel 4950 4150 3    50   Input ~ 0
+Text GLabel 4950 3550 3    50   Input ~ 0
 ~MCLR1
-Wire Wire Line
-	4950 4150 4950 4050
 $Comp
 L power:+5V #PWR0136
 U 1 1 5D0D2792
-P 5050 4550
-F 0 "#PWR0136" H 5050 4400 50  0001 C CNN
-F 1 "+5V" H 5065 4723 50  0000 C CNN
-F 2 "" H 5050 4550 50  0001 C CNN
-F 3 "" H 5050 4550 50  0001 C CNN
-	1    5050 4550
+P 5050 3950
+F 0 "#PWR0136" H 5050 3800 50  0001 C CNN
+F 1 "+5V" H 5065 4123 50  0000 C CNN
+F 2 "" H 5050 3950 50  0001 C CNN
+F 3 "" H 5050 3950 50  0001 C CNN
+	1    5050 3950
 	0    -1   -1   0
 $EndComp
 Wire Wire Line
-	5050 4050 5050 4550
+	5050 3550 5050 3950
 $Comp
 L power:GND #PWR0137
 U 1 1 5D0DC3E9
-P 5150 4400
-F 0 "#PWR0137" H 5150 4150 50  0001 C CNN
-F 1 "GND" H 5155 4227 50  0000 C CNN
-F 2 "" H 5150 4400 50  0001 C CNN
-F 3 "" H 5150 4400 50  0001 C CNN
-	1    5150 4400
-	-1   0    0    -1
-$EndComp
-Wire Wire Line
-	5150 4400 5150 4050
-Wire Wire Line
-	5250 4150 5250 4050
-Wire Wire Line
-	5350 4150 5350 4050
-NoConn ~ 5450 4050
+P 5150 3700
+F 0 "#PWR0137" H 5150 3450 50  0001 C CNN
+F 1 "GND" H 5155 3527 50  0000 C CNN
+F 2 "" H 5150 3700 50  0001 C CNN
+F 3 "" H 5150 3700 50  0001 C CNN
+	1    5150 3700
+	-1   0    0    -1
+$EndComp
+Wire Wire Line
+	5150 3700 5150 3550
+NoConn ~ 5450 3550
 $Comp
 L Connector:Conn_01x06_Male J8
 U 1 1 5D100621
-P 6250 3850
-F 0 "J8" V 6312 4094 50  0000 L CNN
-F 1 "ICSP_Slave" V 6200 3600 50  0000 L CNN
-F 2 "" H 6250 3850 50  0001 C CNN
-F 3 "~" H 6250 3850 50  0001 C CNN
-	1    6250 3850
+P 6250 3350
+F 0 "J8" V 6312 3594 50  0000 L CNN
+F 1 "ICSP_Slave" V 6200 3100 50  0000 L CNN
+F 2 "" H 6250 3350 50  0001 C CNN
+F 3 "~" H 6250 3350 50  0001 C CNN
+	1    6250 3350
 	0    -1   1    0
 $EndComp
-Text GLabel 6450 4150 3    50   Input ~ 0
+Text GLabel 6450 3550 3    50   Input ~ 0
 PGC2
-Text GLabel 6350 4150 3    50   Input ~ 0
+Text GLabel 6350 3550 3    50   Input ~ 0
 PGD2
-Text GLabel 6050 4150 3    50   Input ~ 0
+Text GLabel 6050 3550 3    50   Input ~ 0
 ~MCLR2
-Wire Wire Line
-	6050 4150 6050 4050
 $Comp
 L power:+5V #PWR0138
 U 1 1 5D10062F
-P 6150 4550
-F 0 "#PWR0138" H 6150 4400 50  0001 C CNN
-F 1 "+5V" H 6165 4723 50  0000 C CNN
-F 2 "" H 6150 4550 50  0001 C CNN
-F 3 "" H 6150 4550 50  0001 C CNN
-	1    6150 4550
+P 6150 3950
+F 0 "#PWR0138" H 6150 3800 50  0001 C CNN
+F 1 "+5V" H 6165 4123 50  0000 C CNN
+F 2 "" H 6150 3950 50  0001 C CNN
+F 3 "" H 6150 3950 50  0001 C CNN
+	1    6150 3950
 	0    -1   -1   0
 $EndComp
 Wire Wire Line
-	6150 4050 6150 4550
+	6150 3550 6150 3950
 $Comp
 L power:GND #PWR0139
 U 1 1 5D10063A
-P 6250 4400
-F 0 "#PWR0139" H 6250 4150 50  0001 C CNN
-F 1 "GND" H 6255 4227 50  0000 C CNN
-F 2 "" H 6250 4400 50  0001 C CNN
-F 3 "" H 6250 4400 50  0001 C CNN
-	1    6250 4400
-	-1   0    0    -1
-$EndComp
-Wire Wire Line
-	6250 4400 6250 4050
-Wire Wire Line
-	6350 4150 6350 4050
-Wire Wire Line
-	6450 4150 6450 4050
-NoConn ~ 6550 4050
-Text Notes 5500 5000 0    100  ~ 20
+P 6250 3700
+F 0 "#PWR0139" H 6250 3450 50  0001 C CNN
+F 1 "GND" H 6255 3527 50  0000 C CNN
+F 2 "" H 6250 3700 50  0001 C CNN
+F 3 "" H 6250 3700 50  0001 C CNN
+	1    6250 3700
+	-1   0    0    -1
+$EndComp
+Wire Wire Line
+	6250 3700 6250 3550
+NoConn ~ 6550 3550
+Text Notes 5500 4250 0    100  ~ 20
 ICSP
 Text GLabel 900  3100 0    50   Input ~ 0
@@
 NoConn ~ 1000 6600
 NoConn ~ 1000 6500
-NoConn ~ 1000 6200
 NoConn ~ 1000 6100
 NoConn ~ 1000 5800
@@
 NoConn ~ 1000 4800
 NoConn ~ 1000 4700
+$Comp
+L Connector:Conn_01x02_Male J16
+U 1 1 5D4A8067
+P 5150 4500
+F 0 "J16" V 5212 4544 50  0000 L CNN
+F 1 "Jetson_I2C" V 5100 4250 50  0000 L CNN
+F 2 "" H 5150 4500 50  0001 C CNN
+F 3 "~" H 5150 4500 50  0001 C CNN
+	1    5150 4500
+	0    1    1    0
+$EndComp
+Text GLabel 5150 4800 3    50   Input ~ 0
+SCL
+Text GLabel 5050 4800 3    50   Input ~ 0
+SDA
+Wire Wire Line
+	5150 4800 5150 4700
+Wire Wire Line
+	5050 4700 5050 4800
+Wire Notes Line
+	4400 4300 7000 4300
+Wire Notes Line
+	5800 4300 5800 5400
+$Comp
+L Connector:Conn_01x03_Female J17
+U 1 1 5D4EAFD3
+P 6300 4500
+F 0 "J17" V 6238 4312 50  0000 R CNN
+F 1 "Servo" V 6350 4600 50  0000 R CNN
+F 2 "" H 6300 4500 50  0001 C CNN
+F 3 "~" H 6300 4500 50  0001 C CNN
+	1    6300 4500
+	0    -1   -1   0
+$EndComp
+$Comp
+L power:GND #PWR01
+U 1 1 5D4ECCA1
+P 6400 4750
+F 0 "#PWR01" H 6400 4500 50  0001 C CNN
+F 1 "GND" H 6405 4577 50  0000 C CNN
+F 2 "" H 6400 4750 50  0001 C CNN
+F 3 "" H 6400 4750 50  0001 C CNN
+	1    6400 4750
+	0    -1   1    0
+$EndComp
+Wire Wire Line
+	6400 4750 6400 4700
+Wire Wire Line
+	900  2600 1000 2600
+Text GLabel 900  2600 0    50   Input ~ 0
+PWM1
+Wire Wire Line
+	3800 2900 3700 2900
+Text GLabel 3800 2900 2    50   Input ~ 0
+PWM3
+Wire Wire Line
+	3800 2700 3700 2700
+Text GLabel 3800 2700 2    50   Input ~ 0
+PWM2
+Wire Wire Line
+	900  1600 1000 1600
+Text GLabel 900  1600 0    50   Input ~ 0
+PWM4
+Text GLabel 6300 4700 3    50   Input ~ 0
+BEC3
+Text GLabel 6200 4700 3    50   Input ~ 0
+SERVO
+Text GLabel 900  6200 0    50   Input ~ 0
+SERVO
+Wire Wire Line
+	900  6200 1000 6200
+Text Notes 4600 5350 0    100  ~ 20
+     I2C\nHaberleşmesi
+Text Notes 6050 5350 0    100  ~ 20
+ Servo\nKontrolü
 $EndSCHEMATC

Commit message: Update schematics.
Parts:
- removed J10: UST_1, symbol Connector:Screw_Terminal_01x03
- removed J17: Servo, symbol Connector:Conn_01x03_Female
- removed J3: SOL, symbol Connector:Screw_Terminal_01x03
- removed J4: UST_2, symbol Connector:Screw_Terminal_01x03
- removed J9: SAG, symbol Connector:Screw_Terminal_01x03
- added J21: RS485, symbol Connector:Screw_Terminal_01x02
- added R14, R15, R16: 10k, symbol Device:R
- added R17, R18: 20k, symbol Device:R
- added R19: 120, symbol Device:R
- added U8: MAX485E, symbol Interface_UART:MAX485E
Connections:
- net +5V: now also R14.1, R15.1, R16.1, R18.2, U8.8 (VCC)
- net ENABLE: now also R15.2, U8.2 (~RE), U8.3 (DE)
- net GND: now also R17.1, U8.5 (GND)
- net TX2: now reaches U1.29 (RD6/TX2/CK2/P1C/AN26)
- net TX2: now also R4.2, U5.4 (DI)
- net RX2: now reaches U1.30 (RD7/RX2/DT2/P1D/AN27)
- net RX2: now also R6.2, U5.1 (RO)
- net PWM1: no longer names the net of U1.17 (RC2/CTPLS/CCP1/P1A/T5CKI/AN14)
- net PWM2: no longer names the net of U1.36 (AN9/C12IN2-/CTED2/CCP2/RB3)
- net PWM3: no longer names the net of U1.38 (AN13/CCP3/T1G/IOC/CCP3/RB5)
- net PWM4: no longer names the net of U1.20 (RD1/SDI1/SDA2/CCP4/AN21)
- removed net RX: R6.2, U1.26 (RC7/RX1/DT1/AN19), U5.1 (RO)
- net SERVO: no longer names the net of U2.17 (RC2/CTPLS/CCP1/P1A/T5CKI/AN14)
- removed net TX: R4.2, U1.25 (RC6/TX1/CK1/AN18), U5.4 (DI)
- new net: J21.2 (Pin_2), R18.1, R19.2, U8.6 (A)
- new net: J21.1 (Pin_1), R17.2, R19.1, U8.7 (B)
- new net RX1: R16.2, U1.26 (RC7/RX1/DT1/AN19), U8.1 (RO)
- new net TX1: R14.2, U1.25 (RC6/TX1/CK1/AN18), U8.4 (DI)
- no-connect marks 55 -> 58
Other:
- note added: "Motor Kontrolü"
- note added: "RS-485 Kumanda Haberleşmesi"
- note added: "RS-485 PC Haberleşmesi"
- note removed: "ESC Bağlantıları"
- note removed: "RS-485 Haberleşmesi"
- note removed: "Servo\nKontrolü"
- moved on the sheet: J1, J11, J14, J16, J6, J7, R1, R10, R12, R2, R4, R5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

Commit message: Update schematics.
Changed lines of the file:
@@
 	1550 7350 1800 7350
 Text Label 1800 7250 2    50   ~ 0
-SLC
+SCL
 Text Label 1800 7350 2    50   ~ 0
 SDA

Commit message: Schematic updates.
Parts:
- removed J1, J11, J7: JSN-SR04T, symbol Connector:Conn_01x04_Female
- added R20, R21: 4k7, symbol Device:R_Small
Connections:
- net +5V: now also R20.2, R21.1
- net SCL: now also R21.2
- net SDA: now also R20.1
- net EN1: now reaches U1.2 (AN0/C12IN0-/RA0)
- net EN1: now also R15.2, U8.2 (~RE), U8.3 (DE)
- net ENABLE renamed EN2
- net EN2: no longer R15.2, U8.2 (~RE), U8.3 (DE)
- no-connect marks 58 -> 57
Other:
- note added: "- Motor Kontrolü\n- Sonar Kontrolü"
- note removed: "Motor Kontrolü"
- note removed: "Ultrasonik Sensörler"
- moved on the sheet: R1, R2, U1, U2
