File: Timsah_Main_Board/Timsah_Main_Board.sch (KiCad schematic (older format))
At the start: 48 parts, among them J12 Raspberry_PWR, J13 Jetson_PWR, J14 RS485, J15 PWR_IN, J16 Jetson_I2C, J2 ICSP_Main, J21 RS485, J5 MPU9250, J6 MS5803-14BA, J8 ICSP_Slave, SW1 PWR, U1 PIC18F45K22-IP, U2 PIC18F45K22-IP, U3 AMS1117-3.3, U4 LM338, U5 MAX485E, U6 LM338, U8 MAX485E

Commit message: Added software.
Parts:
- C1, C2, C3, C4: footprint (none) -> Capacitor_THT:CP_Radial_D6.3mm_P2.50mm
- C5, C6: footprint (none) -> Capacitor_THT:CP_Radial_D8.0mm_P3.80mm
- D1: footprint (none) -> LED_THT:LED_D5.0mm
- J16: footprint (none) -> Connector_PinHeader_2.54mm:PinHeader_1x02_P2.54mm_Vertical
- J2, J8: footprint (none) -> Connector_PinHeader_2.54mm:PinHeader_1x06_P2.54mm_Vertical
- J5: footprint (none) -> Connector_PinSocket_2.54mm:PinSocket_1x10_P2.54mm_Vertical
- J6: footprint (none) -> Connector_PinHeader_2.54mm:PinHeader_1x07_P2.54mm_Vertical
- R1, R10, R11, R12, R13, R14, R15, R16, R17, R18, R19, R2, R20, R21, R3, R4, R5, R6, R7, R8, R9: footprint (none) -> Resistor_THT:R_Axial_DIN0207_L6.3mm_D2.5mm_P10.16mm_Horizontal
- U1, U2: footprint Package_DIP:DIP-42_W15.24mm_LongPads -> Package_DIP:DIP-40_W15.24mm_Socket
- U5, U8: footprint (none) -> Package_DIP:DIP-8_W7.62mm_Socket
Changed lines of the file:
@@
 F 0 "U2" H 1250 7100 50  0000 C CNN
 F 1 "PIC18F45K22-IP" H 1500 7000 50  0000 C CNN
-F 2 "Package_DIP:DIP-42_W15.24mm_LongPads" H 2300 5650 50  0001 C CIN
+F 2 "Package_DIP:DIP-40_W15.24mm_Socket" H 2300 5650 50  0001 C CIN
 F 3 "" H 2400 5450 50  0001 C CNN
 	1    2450 5850
@@
 F 0 "R2" V 3900 4800 50  0000 L CNN
 F 1 "10k" V 4100 4750 50  0000 L CNN
-F 2 "" V 3930 4850 50  0001 C CNN
+F 2 "Resistor_THT:R_Axial_DIN0207_L6.3mm_D2.5mm_P10.16mm_Horizontal" V 3930 4850 50  0001 C CNN
 F 3 "~" H 4000 4850 50  0001 C CNN
 	1    4000 4850
@@
 F 0 "J5" V 5765 6830 50  0000 C CNN
 F 1 "MPU9250" V 5674 6830 50  0000 C CNN
-F 2 "" H 5600 6900 50  0001 C CNN
+F 2 "Connector_PinSocket_2.54mm:PinSocket_1x10_P2.54mm_Vertical" H 5600 6900 50  0001 C CNN
 F 3 "~" H 5600 6900 50  0001 C CNN
 	1    5600 6900
@@
 F 0 "R8" H 9020 1646 50  0000 L CNN
 F 1 "820" H 9020 1555 50  0000 L CNN
-F 2 "" V 8880 1600 50  0001 C CNN
+F 2 "Resistor_THT:R_Axial_DIN0207_L6.3mm_D2.5mm_P10.16mm_Horizontal" V 8880 1600 50  0001 C CNN
 F 3 "~" H 8950 1600 50  0001 C CNN
 	1    8950 1600
@@
 F 0 "R7" H 8570 1196 50  0000 L CNN
 F 1 "270" H 8570 1105 50  0000 L CNN
-F 2 "" V 8430 1150 50  0001 C CNN
+F 2 "Resistor_THT:R_Axial_DIN0207_L6.3mm_D2.5mm_P10.16mm_Horizontal" V 8430 1150 50  0001 C CNN
 F 3 "~" H 8500 1150 50  0001 C CNN
 	1    8500 1150
@@
 F 0 "C5" H 9492 1346 50  0000 L CNN
 F 1 "0.1uF" H 9492 1255 50  0000 L CNN
-F 2 "" H 9400 1300 50  0001 C CNN
+F 2 "Capacitor_THT:CP_Radial_D8.0mm_P3.80mm" H 9400 1300 50  0001 C CNN
 F 3 "~" H 9400 1300 50  0001 C CNN
 	1    9400 1300
@@
 F 0 "C2" H 8192 1346 50  0000 L CNN
 F 1 "1uF" H 8192 1255 50  0000 L CNN
-F 2 "" H 8100 1300 50  0001 C CNN
+F 2 "Capacitor_THT:CP_Radial_D6.3mm_P2.50mm" H 8100 1300 50  0001 C CNN
 F 3 "~" H 8100 1300 50  0001 C CNN
 	1    8100 1300
@@
 F 0 "R3" H 7770 1196 50  0000 L CNN
 F 1 "1k" H 7770 1105 50  0000 L CNN
-F 2 "" V 7630 1150 50  0001 C CNN
+F 2 "Resistor_THT:R_Axial_DIN0207_L6.3mm_D2.5mm_P10.16mm_Horizontal" V 7630 1150 50  0001 C CNN
 F 3 "~" H 7700 1150 50  0001 C CNN
 	1    7700 1150
@@
 F 0 "D1" V 7739 1482 50  0000 R CNN
 F 1 "PWR" V 7648 1482 50  0000 R CNN
-F 2 "" H 7700 1600 50  0001 C CNN
+F 2 "LED_THT:LED_D5.0mm" H 7700 1600 50  0001 C CNN
 F 3 "~" H 7700 1600 50  0001 C CNN
 	1    7700 1600
@@
 F 0 "R13" H 10120 3196 50  0000 L CNN
 F 1 "820" H 10120 3105 50  0000 L CNN
-F 2 "" V 9980 3150 50  0001 C CNN
+F 2 "Resistor_THT:R_Axial_DIN0207_L6.3mm_D2.5mm_P10.16mm_Horizontal" V 9980 3150 50  0001 C CNN
 F 3 "~" H 10050 3150 50  0001 C CNN
 	1    10050 3150
@@
 F 0 "R11" H 9670 2746 50  0000 L CNN
 F 1 "270" H 9670 2655 50  0000 L CNN
-F 2 "" V 9530 2700 50  0001 C CNN
+F 2 "Resistor_THT:R_Axial_DIN0207_L6.3mm_D2.5mm_P10.16mm_Horizontal" V 9530 2700 50  0001 C CNN
 F 3 "~" H 9600 2700 50  0001 C CNN
 	1    9600 2700
@@
 F 0 "C6" H 10592 2896 50  0000 L CNN
 F 1 "0.1uF" H 10592 2805 50  0000 L CNN
-F 2 "" H 10500 2850 50  0001 C CNN
+F 2 "Capacitor_THT:CP_Radial_D8.0mm_P3.80mm" H 10500 2850 50  0001 C CNN
 F 3 "~" H 10500 2850 50  0001 C CNN
 	1    10500 2850
@@
 F 0 "C4" H 9292 2896 50  0000 L CNN
 F 1 "1uF" H 9292 2805 50  0000 L CNN
-F 2 "" H 9200 2850 50  0001 C CNN
+F 2 "Capacitor_THT:CP_Radial_D6.3mm_P2.50mm" H 9200 2850 50  0001 C CNN
 F 3 "~" H 9200 2850 50  0001 C CNN
 	1    9200 2850
@@
 F 0 "R1" V 3800 1150 50  0000 L CNN
 F 1 "10k" V 4000 1150 50  0000 L CNN
-F 2 "" V 3830 1200 50  0001 C CNN
+F 2 "Resistor_THT:R_Axial_DIN0207_L6.3mm_D2.5mm_P10.16mm_Horizontal" V 3830 1200 50  0001 C CNN
 F 3 "~" H 3900 1200 50  0001 C CNN
 	1    3900 1200
@@
 F 0 "U1" H 1150 3450 50  0000 C CNN
 F 1 "PIC18F45K22-IP" H 1400 3350 50  0000 C CNN
-F 2 "Package_DIP:DIP-42_W15.24mm_LongPads" H 2200 2000 50  0001 C CIN
+F 2 "Package_DIP:DIP-40_W15.24mm_Socket" H 2200 2000 50  0001 C CIN
 F 3 "" H 2300 1800 50  0001 C CNN
 	1    2350 2200
@@
 F 0 "U5" H 9150 5700 50  0000 C CNN
 F 1 "MAX485E" H 9600 5700 50  0000 C CNN
-F 2 "" H 9400 4550 50  0001 C CNN
+F 2 "Package_DIP:DIP-8_W7.62mm_Socket" H 9400 4550 50  0001 C CNN
 F 3 "https://datasheets.maximintegrated.com/en/ds/MAX1487E-MAX491E.pdf" H 9400 5300 50  0001 C CNN
 	1    9400 5250
@@
 F 0 "R9" H 10020 4946 50  0000 L CNN
 F 1 "20k" H 10020 4855 50  0000 L CNN
-F 2 "" V 9880 4900 50  0001 C CNN
+F 2 "Resistor_THT:R_Axial_DIN0207_L6.3mm_D2.5mm_P10.16mm_Horizontal" V 9880 4900 50  0001 C CNN
 F 3 "~" H 9950 4900 50  0001 C CNN
 	1    9950 4900
@@
 F 0 "R10" H 10020 5746 50  0000 L CNN
 F 1 "20k" H 10020 5655 50  0000 L CNN
-F 2 "" V 9880 5700 50  0001 C CNN
+F 2 "Resistor_THT:R_Axial_DIN0207_L6.3mm_D2.5mm_P10.16mm_Horizontal" V 9880 5700 50  0001 C CNN
 F 3 "~" H 9950 5700 50  0001 C CNN
 	1    9950 5700
@@
 F 0 "R12" H 10270 5346 50  0000 L CNN
 F 1 "120" H 10270 5255 50  0000 L CNN
-F 2 "" V 10130 5300 50  0001 C CNN
+F 2 "Resistor_THT:R_Axial_DIN0207_L6.3mm_D2.5mm_P10.16mm_Horizontal" V 10130 5300 50  0001 C CNN
 F 3 "~" H 10200 5300 50  0001 C CNN
 	1    10200 5300
@@
 F 0 "R5" H 8520 4996 50  0000 L CNN
 F 1 "10k" H 8520 4905 50  0000 L CNN
-F 2 "" V 8380 4950 50  0001 C CNN
+F 2 "Resistor_THT:R_Axial_DIN0207_L6.3mm_D2.5mm_P10.16mm_Horizontal" V 8380 4950 50  0001 C CNN
 F 3 "~" H 8450 4950 50  0001 C CNN
 	1    8450 4950
@@
 F 0 "R6" H 8870 4996 50  0000 L CNN
 F 1 "10k" H 8870 4905 50  0000 L CNN
-F 2 "" V 8730 4950 50  0001 C CNN
+F 2 "Resistor_THT:R_Axial_DIN0207_L6.3mm_D2.5mm_P10.16mm_Horizontal" V 8730 4950 50  0001 C CNN
 F 3 "~" H 8800 4950 50  0001 C CNN
 	1    8800 4950
@@
 F 0 "R4" H 8170 4996 50  0000 L CNN
 F 1 "10k" H 8170 4905 50  0000 L CNN
-F 2 "" V 8030 4950 50  0001 C CNN
+F 2 "Resistor_THT:R_Axial_DIN0207_L6.3mm_D2.5mm_P10.16mm_Horizontal" V 8030 4950 50  0001 C CNN
 F 3 "~" H 8100 4950 50  0001 C CNN
 	1    8100 4950
@@
 F 0 "C1" H 7408 2746 50  0000 R CNN
 F 1 "0.1uF" H 7408 2655 50  0000 R CNN
-F 2 "" H 7500 2700 50  0001 C CNN
+F 2 "Capacitor_THT:CP_Radial_D6.3mm_P2.50mm" H 7500 2700 50  0001 C CNN
 F 3 "~" H 7500 2700 50  0001 C CNN
 	1    7500 2700
@@
 F 0 "C3" H 8208 2746 50  0000 R CNN
 F 1 "1uF" H 8208 2655 50  0000 R CNN
-F 2 "" H 8300 2700 50  0001 C CNN
+F 2 "Capacitor_THT:CP_Radial_D6.3mm_P2.50mm" H 8300 2700 50  0001 C CNN
 F 3 "~" H 8300 2700 50  0001 C CNN
 	1    8300 2700
@@
 F 0 "J6" V 5265 2130 50  0000 C CNN
 F 1 "MS5803-14BA" V 5174 2130 50  0000 C CNN
-F 2 "" H 5100 2150 50  0001 C CNN
+F 2 "Connector_PinHeader_2.54mm:PinHeader_1x07_P2.54mm_Vertical" H 5100 2150 50  0001 C CNN
 F 3 "~" H 5100 2150 50  0001 C CNN
 	1    5100 2150
@@
 F 0 "J2" V 5212 3594 50  0000 L CNN
 F 1 "ICSP_Main" V 5100 3150 50  0000 L CNN
-F 2 "" H 5150 3350 50  0001 C CNN
+F 2 "Connector_PinHeader_2.54mm:PinHeader_1x06_P2.54mm_Vertical" H 5150 3350 50  0001 C CNN
 F 3 "~" H 5150 3350 50  0001 C CNN
 	1    5150 3350
@@
 F 0 "J8" V 6312 3594 50  0000 L CNN
 F 1 "ICSP_Slave" V 6200 3100 50  0000 L CNN
-F 2 "" H 6250 3350 50  0001 C CNN
+F 2 "Connector_PinHeader_2.54mm:PinHeader_1x06_P2.54mm_Vertical" H 6250 3350 50  0001 C CNN
 F 3 "~" H 6250 3350 50  0001 C CNN
 	1    6250 3350
@@
 F 0 "J16" V 6462 2194 50  0000 L CNN
 F 1 "Jetson_I2C" V 6350 1900 50  0000 L CNN
-F 2 "" H 6400 2150 50  0001 C CNN
+F 2 "Connector_PinHeader_2.54mm:PinHeader_1x02_P2.54mm_Vertical" H 6400 2150 50  0001 C CNN
 F 3 "~" H 6400 2150 50  0001 C CNN
 	1    6400 2150
@@
 F 0 "U8" H 5750 5700 50  0000 C CNN
 F 1 "MAX485E" H 6200 5700 50  0000 C CNN
-F 2 "" H 6000 4550 50  0001 C CNN
+F 2 "Package_DIP:DIP-8_W7.62mm_Socket" H 6000 4550 50  0001 C CNN
 F 3 "https://datasheets.maximintegrated.com/en/ds/MAX1487E-MAX491E.pdf" H 6000 5300 50  0001 C CNN
 	1    6000 5250
@@
 F 0 "R17" H 6620 4946 50  0000 L CNN
 F 1 "20k" H 6620 4855 50  0000 L CNN
-F 2 "" V 6480 4900 50  0001 C CNN
+F 2 "Resistor_THT:R_Axial_DIN0207_L6.3mm_D2.5mm_P10.16mm_Horizontal" V 6480 4900 50  0001 C CNN
 F 3 "~" H 6550 4900 50  0001 C CNN
 	1    6550 4900
@@
 F 0 "R18" H 6620 5746 50  0000 L CNN
 F 1 "20k" H 6620 5655 50  0000 L CNN
-F 2 "" V 6480 5700 50  0001 C CNN
+F 2 "Resistor_THT:R_Axial_DIN0207_L6.3mm_D2.5mm_P10.16mm_Horizontal" V 6480 5700 50  0001 C CNN
 F 3 "~" H 6550 5700 50  0001 C CNN
 	1    6550 5700
@@
 F 0 "R19" H 6870 5346 50  0000 L CNN
 F 1 "120" H 6870 5255 50  0000 L CNN
-F 2 "" V 6730 5300 50  0001 C CNN
+F 2 "Resistor_THT:R_Axial_DIN0207_L6.3mm_D2.5mm_P10.16mm_Horizontal" V 6730 5300 50  0001 C CNN
 F 3 "~" H 6800 5300 50  0001 C CNN
 	1    6800 5300
@@
 F 0 "R15" H 5120 4996 50  0000 L CNN
 F 1 "10k" H 5120 4905 50  0000 L CNN
-F 2 "" V 4980 4950 50  0001 C CNN
+F 2 "Resistor_THT:R_Axial_DIN0207_L6.3mm_D2.5mm_P10.16mm_Horizontal" V 4980 4950 50  0001 C CNN
 F 3 "~" H 5050 4950 50  0001 C CNN
 	1    5050 4950
@@
 F 0 "R16" H 5470 4996 50  0000 L CNN
 F 1 "10k" H 5470 4905 50  0000 L CNN
-F 2 "" V 5330 4950 50  0001 C CNN
+F 2 "Resistor_THT:R_Axial_DIN0207_L6.3mm_D2.5mm_P10.16mm_Horizontal" V 5330 4950 50  0001 C CNN
 F 3 "~" H 5400 4950 50  0001 C CNN
 	1    5400 4950
@@
 F 0 "R14" H 4770 4996 50  0000 L CNN
 F 1 "10k" H 4770 4905 50  0000 L CNN
-F 2 "" V 4630 4950 50  0001 C CNN
+F 2 "Resistor_THT:R_Axial_DIN0207_L6.3mm_D2.5mm_P10.16mm_Horizontal" V 4630 4950 50  0001 C CNN
 F 3 "~" H 4700 4950 50  0001 C CNN
 	1    4700 4950
@@
 F 0 "R20" V 6000 2450 50  0000 C CNN
 F 1 "4k7" V 6200 2450 50  0000 C CNN
-F 2 "" H 6100 2450 50  0001 C CNN
+F 2 "Resistor_THT:R_Axial_DIN0207_L6.3mm_D2.5mm_P10.16mm_Horizontal" H 6100 2450 50  0001 C CNN
 F 3 "~" H 6100 2450 50  0001 C CNN
 	1    6100 2450
@@
 F 0 "R21" V 6500 2450 50  0000 C CNN
 F 1 "4k7" V 6700 2450 50  0000 C CNN
-F 2 "" H 6600 2450 50  0001 C CNN
+F 2 "Resistor_THT:R_Axial_DIN0207_L6.3mm_D2.5mm_P10.16mm_Horizontal" H 6600 2450 50  0001 C CNN
 F 3 "~" H 6600 2450 50  0001 C CNN
 	1    6600 2450

Commit message: Hardware Update
Parts:
- removed C3, C4: 1uF, Capacitor_THT:CP_Radial_D6.3mm_P2.50mm, symbol Device:C_Small
- removed C6: 0.1uF, Capacitor_THT:CP_Radial_D8.0mm_P3.80mm, symbol Device:C_Small
- removed F2: 5A, symbol Device:Fuse
- removed J12: Raspberry_PWR, symbol Connector:Screw_Terminal_01x03
- removed J13: Jetson_PWR, symbol Connector:Screw_Terminal_01x03
- removed J2: ICSP_Main, Connector_PinHeader_2.54mm:PinHeader_1x06_P2.54mm_Vertical, symbol Connector:Conn_01x06_Male
- removed J8: ICSP_Slave, Connector_PinHeader_2.54mm:PinHeader_1x06_P2.54mm_Vertical, symbol Connector:Conn_01x06_Male
- removed R11: 270, Resistor_THT:R_Axial_DIN0207_L6.3mm_D2.5mm_P10.16mm_Horizontal, symbol Device:R
- removed R13: 820, Resistor_THT:R_Axial_DIN0207_L6.3mm_D2.5mm_P10.16mm_Horizontal, symbol Device:R
- removed U3: AMS1117-3.3, Package_TO_SOT_SMD:SOT-223-3_TabPin2, symbol Regulator_Linear:AMS1117-3.3
- removed U6: LM338, Package_TO_SOT_THT:TO-3, symbol Symols:LM338
- added C2: 1uF, Capacitor_SMD:C_0805_2012Metric_Pad1.15x1.40mm_HandSolder, symbol Device:C_Small
- added C5: 10uF, Capacitor_SMD:C_0805_2012Metric_Pad1.15x1.40mm_HandSolder, symbol Device:C
- added J10: Jetson_GROUND, TerminalBlock_4Ucon:TerminalBlock_4Ucon_1x02_P3.50mm_Vertical, symbol Connector:Screw_Terminal_01x02
- added J2: ICSP_Main, Connector_PinSocket_2.54mm:PinSocket_1x05_P2.54mm_Vertical, symbol Connector:Conn_01x05_Male
- added J4: ICSP_Slave, Connector_PinSocket_2.54mm:PinSocket_1x05_P2.54mm_Vertical, symbol Connector:Conn_01x05_Male
- added J7: Raspberry_PWR, TerminalBlock_4Ucon:TerminalBlock_4Ucon_1x02_P3.50mm_Vertical, symbol Connector:Screw_Terminal_01x02
- added J8: Raspberry_GROUN, TerminalBlock_4Ucon:TerminalBlock_4Ucon_1x02_P3.50mm_Vertical, symbol Connector:Screw_Terminal_01x02
- added J9: Jetson_PWR, TerminalBlock_4Ucon:TerminalBlock_4Ucon_1x02_P3.50mm_Vertical, symbol Connector:Screw_Terminal_01x02
- C1: value 0.1uF -> 1uF; footprint Capacitor_THT:CP_Radial_D6.3mm_P2.50mm -> Capacitor_SMD:C_0805_2012Metric_Pad1.15x1.40mm_HandSolder
- C3: renamed from C2; footprint Capacitor_THT:CP_Radial_D6.3mm_P2.50mm -> Capacitor_SMD:C_0805_2012Metric_Pad1.15x1.40mm_HandSolder
- C4: renamed from C5; footprint Capacitor_THT:CP_Radial_D8.0mm_P3.80mm -> Capacitor_SMD:C_0805_2012Metric_Pad1.15x1.40mm_HandSolder
- D1: footprint LED_THT:LED_D5.0mm -> LED_SMD:LED_0805_2012Metric_Pad1.15x1.40mm_HandSolder
- F1: footprint (none) -> Footprints:Fuseholder_23x9x10mm
- J1: renamed from J6; footprint Connector_PinHeader_2.54mm:PinHeader_1x07_P2.54mm_Vertical -> Connector_PinSocket_2.54mm:PinSocket_1x07_P2.54mm_Vertical
- J11: renamed from J15; footprint (none) -> TerminalBlock:TerminalBlock_bornier-2_P5.08mm
- J12: renamed from J14; footprint (none) -> TerminalBlock_4Ucon:TerminalBlock_4Ucon_1x02_P3.50mm_Vertical
- J3: renamed from J5; value MPU9250 -> BNO055; footprint Connector_PinSocket_2.54mm:PinSocket_1x10_P2.54mm_Vertical -> Footprints:BNO055-Module_Adafruit
- J6: renamed from J21; footprint (none) -> TerminalBlock_4Ucon:TerminalBlock_4Ucon_1x02_P3.50mm_Vertical
- R1, R2: footprint Resistor_THT:R_Axial_DIN0207_L6.3mm_D2.5mm_P10.16mm_Horizontal -> Resistor_SMD:R_0805_2012Metric_Pad1.15x1.40mm_HandSolder
- R11: renamed from R3; footprint Resistor_THT:R_Axial_DIN0207_L6.3mm_D2.5mm_P10.16mm_Horizontal -> Resistor_SMD:R_0805_2012Metric_Pad1.15x1.40mm_HandSolder
- R12: renamed from R4; footprint Resistor_THT:R_Axial_DIN0207_L6.3mm_D2.5mm_P10.16mm_Horizontal -> Resistor_SMD:R_0805_2012Metric_Pad1.15x1.40mm_HandSolder
- R14: renamed from R5; footprint Resistor_THT:R_Axial_DIN0207_L6.3mm_D2.5mm_P10.16mm_Horizontal -> Resistor_SMD:R_0805_2012Metric_Pad1.15x1.40mm_HandSolder
- R15: renamed from R6; footprint Resistor_THT:R_Axial_DIN0207_L6.3mm_D2.5mm_P10.16mm_Horizontal -> Resistor_SMD:R_0805_2012Metric_Pad1.15x1.40mm_HandSolder
- R17: renamed from R9; footprint Resistor_THT:R_Axial_DIN0207_L6.3mm_D2.5mm_P10.16mm_Horizontal -> Resistor_SMD:R_0805_2012Metric_Pad1.15x1.40mm_HandSolder
- R18: renamed from R10; footprint Resistor_THT:R_Axial_DIN0207_L6.3mm_D2.5mm_P10.16mm_Horizontal -> Resistor_SMD:R_0805_2012Metric_Pad1.15x1.40mm_HandSolder
- R3: renamed from R14; footprint Resistor_THT:R_Axial_DIN0207_L6.3mm_D2.5mm_P10.16mm_Horizontal -> Resistor_SMD:R_0805_2012Metric_Pad1.15x1.40mm_HandSolder
- R4: renamed from R15; footprint Resistor_THT:R_Axial_DIN0207_L6.3mm_D2.5mm_P10.16mm_Horizontal -> Resistor_SMD:R_0805_2012Metric_Pad1.15x1.40mm_HandSolder
- R5: renamed from R16; footprint Resistor_THT:R_Axial_DIN0207_L6.3mm_D2.5mm_P10.16mm_Horizontal -> Resistor_SMD:R_0805_2012Metric_Pad1.15x1.40mm_HandSolder
- R6: renamed from R20; footprint Resistor_THT:R_Axial_DIN0207_L6.3mm_D2.5mm_P10.16mm_Horizontal -> Resistor_SMD:R_0805_2012Metric_Pad1.15x1.40mm_HandSolder
- R7: renamed from R17; footprint Resistor_THT:R_Axial_DIN0207_L6.3mm_D2.5mm_P10.16mm_Horizontal -> Resistor_SMD:R_0805_2012Metric_Pad1.15x1.40mm_HandSolder
- R8: renamed from R18; footprint Resistor_THT:R_Axial_DIN0207_L6.3mm_D2.5mm_P10.16mm_Horizontal -> Resistor_SMD:R_0805_2012Metric_Pad1.15x1.40mm_HandSolder
- R9: renamed from R21; footprint Resistor_THT:R_Axial_DIN0207_L6.3mm_D2.5mm_P10.16mm_Horizontal -> Resistor_SMD:R_0805_2012Metric_Pad1.15x1.40mm_HandSolder
- SW1: footprint (none) -> Footprints:SW_Slide_1P2T_0.105pitch
- renumbered J16 to J5, R19 to R10, R7 to R13, R8 to R16, R12 to R19, U8 to U3
Connections:
- net +3V3: now also J1.6 (Pin_6), J3.2 (Pin_2); no longer C1.1
- net +5V: now also C1.1, J3.1 (Pin_1), C2.1, C5.1, J2.2 (Pin_2), J4.2 (Pin_2); no longer J3.10 (Pin_10), U1.11 (VDD), U1.32 (VDD), U2.11 (VDD), U2.32 (VDD)
- net GND: now also J3.3 (Pin_3), C2.2, C5.2, J10.1 (Pin_1), J10.2 (Pin_2), J2.3 (Pin_3), J4.3 (Pin_3), J8.1 (Pin_1), J8.2 (Pin_2); no longer J1.6 (Pin_6), J3.1 (Pin_1), J3.4 (Pin_4), J3.9 (Pin_9)
- net INT: now also J3.8 (Pin_8); no longer J3.3 (Pin_3)
- net PGC1: now also J2.5 (Pin_5)
- net PGC2: now also J4.5 (Pin_5)
- net PGD1: now also J2.4 (Pin_4)
- net PGD2: now also J4.4 (Pin_4)
- net RX1: now also U1.30 (RD7/RX2/DT2/P1D/AN27); no longer U1.26 (RC7/RX1/DT1/AN19)
- net RX2: now also U1.26 (RC7/RX1/DT1/AN19); no longer U1.30 (RD7/RX2/DT2/P1D/AN27)
- net SCL: now also J1.4 (Pin_4), J3.5 (Pin_5); no longer J3.8 (Pin_8)
- net SDA: now also J1.3 (Pin_3), J3.4 (Pin_4); no longer J3.7 (Pin_7)
- net TX1: now also U1.29 (RD6/TX2/CK2/P1C/AN26); no longer U1.25 (RC6/TX1/CK1/AN18)
- net TX2: now also U1.25 (RC6/TX1/CK1/AN18); no longer U1.29 (RD6/TX2/CK2/P1C/AN26)
- net ~MCLR1: now also J2.1 (Pin_1)
- net ~MCLR2: now also J4.1 (Pin_1)
- net UL-R: now reaches U1.33 (AN12/SRI/FLT0/INT0/RB0)
- net UR-R: now reaches U1.34 (AN10/C12IN3-/INT1/RB1)
- net BL-R: now reaches U1.35 (AN8/CTED1/INT2/RB2)
- net BR-R: now reaches U1.36 (AN9/C12IN2-/CTED2/CCP2/RB3)
- net RST: now reaches J3.6 (Pin_6)
- net +12V: now reaches J11.1 (Pin_1), SW1.2 (B)
- net 5V-NANO renamed +5VD
- net +5VD: now also J7.1 (Pin_1), J7.2 (Pin_2), J9.1 (Pin_1), J9.2 (Pin_2)
- net SCL2: no longer names the net of U2.19 (RD0/SCL2/SCK2/AN20)
- net SCL2: no longer J1.4 (Pin_4)
- net SDA2: no longer names the net of U2.20 (RD1/SDI1/SDA2/CCP4/AN21)
- net SDA2: no longer J1.3 (Pin_3)
- new net ADR: J3.7 (Pin_7)
- new net BEC4: U1.11 (VDD), U1.32 (VDD)
- new net BEC5: U2.11 (VDD), U2.32 (VDD)
- new net PS0: J3.10 (Pin_10)
- new net PS1: J3.9 (Pin_9)
- no-connect marks 57 -> 52
Other:
- note added: "- Motor Control\n- Sonar Control\n- BLDC Control"
- note added: "9 Axis MEMS Sensor"
- note added: "I2C\nCommunication"
- note added: "Main Microcontroller"
- note added: "Power"
- note added: "Power Out"
- note added: "Pressure Sensor"
- note added: "RS-485 PC Communication"
- note added: "RS-485 Remote Controller Communication"
- note added: "Slave Microcontroller"
- note removed: "- Motor Kontrolü\n- Sonar Kontrolü"
- note removed: "9 Eksen MEMS Sensörü"
- note removed: "Ana Mikrodenetleyici"
- note removed: "Basınç Sensörü"
- note removed: "Güç"
- note removed: "Güç Çıkışı"
- note removed: "I2C\nHaberleşmesi"
- note removed: "RS-485 Kumanda Haberleşmesi"
- note removed: "RS-485 PC Haberleşmesi"
- note removed: "Yardımcı Mikrodenetleyici"
- moved on the sheet: C3, C4, D1, F1, J11, J3, R11, R13, R16, SW1, U4
