File: Timsah_Main_Board/Timsah_Main_Board.sch (KiCad schematic (older format))
At the start: 44 parts, among them J1 MS5803-14BA, J10 Jetson_GROUND, J11 PWR_IN, J12 RS485, J2 ICSP_Main, J3 BNO055, J4 ICSP_Slave, J5 Jetson_I2C, J6 RS485, J7 Raspberry_PWR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

Commit message: Update
Connections:
- net BEC4 is gone; now on net +5V: U1.11 (VDD), U1.32 (VDD)
- net BEC5 is gone; now on net +5V: U2.11 (VDD), U2.32 (VDD)
