File: Timsah_Main_Board/Motor-Controle.sch (KiCad schematic (older format))
At the start: 9 parts, among them J10 SAĞ ARKA, J17 SOL ARKA, J18 SERVO Gripper, J19 SAĞ ÜST, J20 SOL ÜST, J3 SERVO Camera, J4 SAĞ ÖN, J9 SOL ÖN, U7 PCA9685PW

Commit message: Schematic updates.
Parts:
- added J22, J23, J24, J25: JSN-SR04T, symbol Connector:Conn_01x04_Female
Connections:
- net GND: now also J22.4 (Pin_4), J23.4 (Pin_4), J24.4 (Pin_4), J25.4 (Pin_4)
- new net +5V: J22.1 (Pin_1), J23.1 (Pin_1), J24.1 (Pin_1), J25.1 (Pin_1)
- new net ECHO1: J22.3 (Pin_3)
- new net ECHO2: J23.3 (Pin_3)
- new net ECHO3: J24.3 (Pin_3), J25.3 (Pin_3)
- new net TRIG1: J22.2 (Pin_2)
- new net TRIG2: J23.2 (Pin_2)
- new net TRIG3: J24.2 (Pin_2), J25.2 (Pin_2)
Other:
- note added: "Ultrasonik Sensörler"
- moved on the sheet: J18, J3

Commit message: Added software.
Parts:
- J18, J3: footprint (none) -> Connector_PinHeader_2.54mm:PinHeader_1x03_P2.54mm_Vertical
- J22, J23, J24, J25: footprint (none) -> Connector_PinHeader_2.54mm:PinHeader_1x04_P2.54mm_Vertical
Changed lines of the file:
@@
 F 0 "J3" H 3850 2450 50  0000 C CNN
 F 1 "SERVO Camera" H 4000 2000 50  0000 C CNN
-F 2 "" H 3750 2200 50  0001 C CNN
+F 2 "Connector_PinHeader_2.54mm:PinHeader_1x03_P2.54mm_Vertical" H 3750 2200 50  0001 C CNN
 F 3 "~" H 3750 2200 50  0001 C CNN
 	1    3750 2200
@@
 F 0 "J18" H 5550 2450 50  0000 C CNN
 F 1 "SERVO Gripper" H 5700 2000 50  0000 C CNN
-F 2 "" H 5450 2200 50  0001 C CNN
+F 2 "Connector_PinHeader_2.54mm:PinHeader_1x03_P2.54mm_Vertical" H 5450 2200 50  0001 C CNN
 F 3 "~" H 5450 2200 50  0001 C CNN
 	1    5450 2200
@@
 F 0 "J22" H 3950 3500 50  0000 L CNN
 F 1 "JSN-SR04T" H 3850 3350 50  0000 L CNN
-F 2 "" H 4150 3150 50  0001 C CNN
+F 2 "Connector_PinHeader_2.54mm:PinHeader_1x04_P2.54mm_Vertical" H 4150 3150 50  0001 C CNN
 F 3 "~" H 4150 3150 50  0001 C CNN
 	1    4150 3150
@@
 F 0 "J23" H 4700 3500 50  0000 L CNN
 F 1 "JSN-SR04T" H 4600 3350 50  0000 L CNN
-F 2 "" H 4900 3150 50  0001 C CNN
+F 2 "Connector_PinHeader_2.54mm:PinHeader_1x04_P2.54mm_Vertical" H 4900 3150 50  0001 C CNN
 F 3 "~" H 4900 3150 50  0001 C CNN
 	1    4900 3150
@@
 F 0 "J24" H 5450 3500 50  0000 L CNN
 F 1 "JSN-SR04T" H 5350 3350 50  0000 L CNN
-F 2 "" H 5650 3150 50  0001 C CNN
+F 2 "Connector_PinHeader_2.54mm:PinHeader_1x04_P2.54mm_Vertical" H 5650 3150 50  0001 C CNN
 F 3 "~" H 5650 3150 50  0001 C CNN
 	1    5650 3150
@@
 F 0 "J25" H 6200 3500 50  0000 L CNN
 F 1 "JSN-SR04T" H 6100 3350 50  0000 L CNN
-F 2 "" H 6400 3150 50  0001 C CNN
+F 2 "Connector_PinHeader_2.54mm:PinHeader_1x04_P2.54mm_Vertical" H 6400 3150 50  0001 C CNN
 F 3 "~" H 6400 3150 50  0001 C CNN
 	1    6400 3150

Commit message: Hardware Update
Parts:
- removed J25: JSN-SR04T, Connector_PinHeader_2.54mm:PinHeader_1x04_P2.54mm_Vertical, symbol Connector:Conn_01x04_Female
- added J24: Power, TerminalBlock:TerminalBlock_bornier-2_P5.08mm, symbol Connector:Screw_Terminal_01x02
- added J25: Relay Up, Connector_PinSocket_2.54mm:PinSocket_1x02_P2.54mm_Vertical, symbol Connector:Screw_Terminal_01x02
- added J26: Relay Back, Connector_PinSocket_2.54mm:PinSocket_1x02_P2.54mm_Vertical, symbol Connector:Screw_Terminal_01x02
- J14: renamed from J4; footprint (none) -> Connector_PinHeader_2.54mm:PinHeader_1x03_P2.54mm_Vertical
- J15: renamed from J9; footprint (none) -> Connector_PinHeader_2.54mm:PinHeader_1x03_P2.54mm_Vertical
- J16: renamed from J22; footprint Connector_PinHeader_2.54mm:PinHeader_1x04_P2.54mm_Vertical -> Connector_PinSocket_2.54mm:PinSocket_1x04_P2.54mm_Vertical
- J17: renamed from J10; footprint (none) -> Connector_PinHeader_2.54mm:PinHeader_1x03_P2.54mm_Vertical
- J18: renamed from J17; footprint (none) -> Connector_PinHeader_2.54mm:PinHeader_1x03_P2.54mm_Vertical
- J19: renamed from J23; footprint Connector_PinHeader_2.54mm:PinHeader_1x04_P2.54mm_Vertical -> Connector_PinSocket_2.54mm:PinSocket_1x04_P2.54mm_Vertical
- J21: renamed from J24; footprint Connector_PinHeader_2.54mm:PinHeader_1x04_P2.54mm_Vertical -> Connector_PinSocket_2.54mm:PinSocket_1x04_P2.54mm_Vertical
- J22: renamed from J19; footprint (none) -> Connector_PinHeader_2.54mm:PinHeader_1x03_P2.54mm_Vertical
- J23: renamed from J20; footprint (none) -> Connector_PinHeader_2.54mm:PinHeader_1x03_P2.54mm_Vertical
- renumbered J3 to J13, J18 to J20, U7 to U6
Connections:
- net BEC1 is gone; now on net +5V: J13.2 (Pin_2), J14.2 (Pin_2)
- net BEC2 is gone; now on net +5V: J17.2 (Pin_2), J20.2 (Pin_2)
- net BEC3 is gone; now on net +5V: J22.2 (Pin_2), U6.28 (VDD)
- net BEC4 is gone; now on net +5V: J15.2 (Pin_2)
- net BEC5 is gone; now on net +5V: J18.2 (Pin_2)
- net BEC6 is gone; now on net +5V: J23.2 (Pin_2)
- net GND: now also J24.2 (Pin_2)
- new net +12V: J24.1 (Pin_1)
- new net BL-R: J26.2 (Pin_2)
- new net BR-R: J26.1 (Pin_1)
- new net UL-R: J25.2 (Pin_2)
- new net UR-R: J25.1 (Pin_1)
Other:
- note added: "BLDC Control"
- note added: "Connect BEC to 5V"
- note added: "ESC Control"
- note added: "PWM Module"
- note added: "Servo Control"
- note added: "Ultrasonic Sensor"
- note removed: "ESC Kontrolü"
- note removed: "PWM Modülü"
- note removed: "Servo Kontrolü"
- note removed: "Ultrasonik Sensörler"
- moved on the sheet: J16, J19, J21

Commit message: Update
Parts:
- removed J13: SERVO Camera, Connector_PinHeader_2.54mm:PinHeader_1x03_P2.54mm_Vertical, symbol Connector:Conn_01x03_Male
- removed J14: SAĞ ÖN, Connector_PinHeader_2.54mm:PinHeader_1x03_P2.54mm_Vertical, symbol Connector:Screw_Terminal_01x03
- removed J15: SOL ÖN, Connector_PinHeader_2.54mm:PinHeader_1x03_P2.54mm_Vertical, symbol Connector:Screw_Terminal_01x03
- removed J17: SAĞ ARKA, Connector_PinHeader_2.54mm:PinHeader_1x03_P2.54mm_Vertical, symbol Connector:Screw_Terminal_01x03
- removed J18: SOL ARKA, Connector_PinHeader_2.54mm:PinHeader_1x03_P2.54mm_Vertical, symbol Connector:Screw_Terminal_01x03
- removed J20: SERVO Gripper, Connector_PinHeader_2.54mm:PinHeader_1x03_P2.54mm_Vertical, symbol Connector:Conn_01x03_Male
- removed J22: SAĞ ÜST, Connector_PinHeader_2.54mm:PinHeader_1x03_P2.54mm_Vertical, symbol Connector:Screw_Terminal_01x03
- removed J23: SOL ÜST, Connector_PinHeader_2.54mm:PinHeader_1x03_P2.54mm_Vertical, symbol Connector:Screw_Terminal_01x03
- removed U6: PCA9685PW, Package_SO:TSSOP-28_4.4x9.7mm_P0.65mm, symbol Driver_LED:PCA9685PW
- added J19: BEC, TerminalBlock_4Ucon:TerminalBlock_4Ucon_1x02_P3.50mm_Vertical, symbol Connector:Screw_Terminal_01x02
- added J20: PCA9685, Connector_PinSocket_2.54mm:PinSocket_1x06_P2.54mm_Vertical, symbol Connector:Conn_01x06_Female
- renumbered J16 to J13, J24 to J14, J25 to J15, J26 to J16, J19 to J17, J21 to J18
Connections:
- net +5V: now also J19.2 (Pin_2), J20.5 (Pin_5), J20.6 (Pin_6)
- net GND: now also J19.1 (Pin_1), J20.1 (Pin_1), J20.2 (Pin_2)
- net SCL: now also J20.3 (Pin_3)
- net SDA: now also J20.4 (Pin_4)
- no-connect marks 9 -> 0
Other:
- note added: "BEC Power"
- note added: "PCA9685 Module"
- note removed: "Connect BEC to 5V"
- note removed: "ESC Control"
- note removed: "PWM Module"
- note removed: "Servo Control"
- moved on the sheet: J13, J14, J15, J16, J17, J18
