File: Timsah_Main_Board/Timsah_Main_Board.kicad_pcb (KiCad board)
At the start: 2 copper layers, 100 x 100 mm, 59 parts, among them J1 MS5803-14BA, J10 Jetson_GROUND, J11 PWR_IN, J12 RS485, J13 SERVO Camera, J14 SAĞ ÖN, J15 SOL ÖN, J16 JSN-SR04T, J17 SAĞ ARKA, J18 SOL ARKA, J19 JSN-SR04T, J2 ICSP_Main, J20 SERVO Gripper, J21 JSN-SR04T, J22 SAĞ ÜST, J23 SOL ÜST, J24 Power, J25 Relay Up, J26 Relay Back, J3 BNO055, J4 ICSP_Slave, J5 Jetson_I2C, J6 RS485, J7 Raspberry_PWR, J8 Raspberry_GROUN, J9 Jetson_PWR, SW1 PWR, U1 PIC18F45K22-IP, U2 PIC18F45K22-IP, U3 MAX485E, U4 LM338, U5 MAX485E, U6 PCA9685PW

Commit message: Update PCB
Parts:
- moved R17 0.60 mm to (102.6, 110.0)
Routing:
- net GND: track 0.00 -> 457.9 mm, vias 0 -> 3
- net BEC1: track 0.00 -> 325.6 mm, vias 0 -> 5
- net /SCL: track 0.00 -> 165.3 mm, vias 0 -> 6
- net /SDA: track 0.00 -> 137.8 mm, vias 0 -> 4
- net +5VD: track 0.00 -> 95.9 mm
- net EN1: track 0.00 -> 75.5 mm, vias 0 -> 1
- net Net-(C4-Pad1): track 0.00 -> 56.3 mm
- net Net-(R13-Pad2): track 0.00 -> 52.6 mm
- net ECHO3: track 0.00 -> 49.5 mm
- net EN2: track 0.00 -> 44.2 mm
- net Net-(J6-Pad1): track 0.00 -> 35.5 mm
- net +12V: track 0.00 -> 33.1 mm
- net ECHO1: track 0.00 -> 31.3 mm, vias 0 -> 1
- net +3V3: track 0.00 -> 30.3 mm, vias 0 -> 1
- net Net-(J12-Pad2): track 0.00 -> 29.2 mm
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- added copper zone on B.Cu, net GND
- added copper zone on F.Cu, net GND
Other:
- outline, holes or cut-outs redrawn

Commit message: Update
Parts:
- removed J21: JSN-SR04T, Connector_PinSocket_2.54mm:PinSocket_1x04_P2.54mm_Vertical
- removed J22: SAĞ ÜST, Connector_PinHeader_2.54mm:PinHeader_1x03_P2.54mm_Vertical
- removed J23: SOL ÜST, Connector_PinHeader_2.54mm:PinHeader_1x03_P2.54mm_Vertical
- removed J24: Power, TerminalBlock:TerminalBlock_bornier-2_P5.08mm
- removed J25: Relay Up, Connector_PinSocket_2.54mm:PinSocket_1x02_P2.54mm_Vertical
- removed J26: Relay Back, Connector_PinSocket_2.54mm:PinSocket_1x02_P2.54mm_Vertical
- removed U6: PCA9685PW, Package_SO:TSSOP-28_4.4x9.7mm_P0.65mm
- C2, J3, J5, R1, R4, R6, R9: moved to B.Cu
- D1, J12, J6, R10, R11, R13, R16, R19, SW1, U5: moved to F.Cu
- J13: value SERVO Camera -> JSN-SR04T; footprint Connector_PinHeader_2.54mm:PinHeader_1x03_P2.54mm_Vertical -> Connector_PinSocket_2.54mm:PinSocket_1x04_P2.54mm_Vertical; moved to B.Cu
- J14: value SAĞ ÖN -> Power; footprint Connector_PinHeader_2.54mm:PinHeader_1x03_P2.54mm_Vertical -> TerminalBlock:TerminalBlock_bornier-2_P5.08mm; moved to B.Cu
- J15: value SOL ÖN -> Relay Up; footprint Connector_PinHeader_2.54mm:PinHeader_1x03_P2.54mm_Vertical -> Connector_PinSocket_2.54mm:PinSocket_1x02_P2.54mm_Vertical; moved to B.Cu
- J16: value JSN-SR04T -> Relay Back; footprint Connector_PinSocket_2.54mm:PinSocket_1x04_P2.54mm_Vertical -> Connector_PinSocket_2.54mm:PinSocket_1x02_P2.54mm_Vertical
- J17: value SAĞ ARKA -> JSN-SR04T; footprint Connector_PinHeader_2.54mm:PinHeader_1x03_P2.54mm_Vertical -> Connector_PinSocket_2.54mm:PinSocket_1x04_P2.54mm_Vertical; moved to B.Cu
- J18: value SOL ARKA -> JSN-SR04T; footprint Connector_PinHeader_2.54mm:PinHeader_1x03_P2.54mm_Vertical -> Connector_PinSocket_2.54mm:PinSocket_1x04_P2.54mm_Vertical; moved to B.Cu
- J19: value JSN-SR04T -> BEC; footprint Connector_PinSocket_2.54mm:PinSocket_1x04_P2.54mm_Vertical -> TerminalBlock_4Ucon:TerminalBlock_4Ucon_1x02_P3.50mm_Vertical; moved to F.Cu
- J20: value SERVO Gripper -> PCA9685; footprint Connector_PinHeader_2.54mm:PinHeader_1x03_P2.54mm_Vertical -> Connector_PinSocket_2.54mm:PinSocket_1x06_P2.54mm_Vertical
- moved J20 88.4 mm to (145.1, 89.7), turned to 0 degrees
- moved C5 80.6 mm to (141.4, 85.8)
- moved J10 75.5 mm to (137.1, 80.6)
- moved J17 67.3 mm to (121.2, 119.0)
- moved J14 65.2 mm to (116.3, 75.0)
- moved J13 64.3 mm to (121.2, 124.3), turned to 180 degrees
- moved J7 62.0 mm to (63.4, 73.7), turned to 0 degrees
- moved J8 59.4 mm to (73.2, 73.5), turned to 0 degrees
- moved J18 58.8 mm to (121.2, 98.7), turned to 180 degrees
- moved J9 54.6 mm to (127.6, 74.4), turned to 0 degrees
- moved R6 54.1 mm to (140.9, 103.3)
- moved R19 51.8 mm to (58.5, 110.2), turned to 0 degrees
- moved J6 50.8 mm to (136.2, 119.1)
- moved J16 50.0 mm to (80.6, 95.5), turned to 180 degrees
- moved R9 49.5 mm to (140.9, 100.6), turned to 180 degrees
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Connections:
- C1 pad 1: BEC1 -> BEC
- C2 pad 1: BEC1 -> BEC
- C5 pad 1: BEC1 -> BEC
- J13 pad 1: /Motor Controle/SERVO_CAMERA -> BEC
- J13 pad 2: BEC1 -> TRIG1
- J13 pad 3: GND -> ECHO1
- J14 pad 1: /Motor Controle/PWM_FR -> +12V
- J14 pad 2: BEC1 -> GND
- J15 pad 1: /Motor Controle/PWM_FL -> UR-R
- J15 pad 2: BEC1 -> UL-R
- J16 pad 1: BEC1 -> BR-R
- J16 pad 2: TRIG1 -> BL-R
- J17 pad 1: /Motor Controle/PWM_BR -> BEC
- J17 pad 2: BEC1 -> TRIG2
- J17 pad 3: GND -> ECHO2
- J18 pad 1: /Motor Controle/PWM_BL -> BEC
- J18 pad 2: BEC1 -> TRIG3
- J18 pad 3: GND -> ECHO3
- J19 pad 1: BEC1 -> GND
- J19 pad 2: TRIG2 -> BEC
- J2 pad 2: BEC1 -> BEC
- J20 pad 1: /Motor Controle/SERVO_GRIPPER -> GND
- J20 pad 2: BEC1 -> GND
- J20 pad 3: GND -> /SCL
- J3 pad 1: BEC1 -> BEC
- J4 pad 2: BEC1 -> BEC
- R1 pad 1: BEC1 -> BEC
- R12 pad 1: BEC1 -> BEC
- R14 pad 1: BEC1 -> BEC
- R15 pad 1: BEC1 -> BEC
- R18 pad 2: BEC1 -> BEC
- R2 pad 1: BEC1 -> BEC
- R3 pad 1: BEC1 -> BEC
- R4 pad 1: BEC1 -> BEC
- R5 pad 1: BEC1 -> BEC
- R6 pad 2: BEC1 -> BEC
- R8 pad 2: BEC1 -> BEC
- R9 pad 1: BEC1 -> BEC
- U1 pad 11: BEC1 -> BEC
- U1 pad 32: BEC1 -> BEC
- U2 pad 11: BEC1 -> BEC
- U2 pad 32: BEC1 -> BEC
- U3 pad 8: BEC1 -> BEC
- U5 pad 8: BEC1 -> BEC
Routing:
- net GND: track 457.9 -> 19.5 mm, vias 3 -> 4
- net BEC1: track 325.6 -> 0.00 mm, vias 5 -> 0
- net BEC: track 0.00 -> 270.2 mm, vias 0 -> 1
- net Net-(J12-Pad1): track 23.3 -> 88.0 mm
- net Net-(J6-Pad2): track 22.2 -> 82.3 mm, vias 0 -> 2
- net Net-(J12-Pad2): track 29.2 -> 78.5 mm
- net Net-(J6-Pad1): track 35.5 -> 78.5 mm, vias 0 -> 2
- net ECHO3: track 49.5 -> 19.7 mm
- net EN2: track 44.2 -> 70.4 mm
- net /Motor Controle/PWM_UL: track 25.1 -> 0.00 mm, vias 4 -> 0
- net /SDA: track 137.8 -> 162.7 mm, vias 4 -> 2
- net ECHO1: track 31.3 -> 8.97 mm, vias 1 -> 0
- net /Motor Controle/PWM_BR: track 21.7 -> 0.00 mm, vias 2 -> 0
- net Net-(R13-Pad2): track 52.6 -> 32.7 mm
- net TRIG1: track 20.9 -> 40.7 mm, vias 0 -> 1
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Other:
- net class Default: trace_width 0.25 -> 0.3
- board text added: "BTU - ROV Timsah 28.08.2019"
